File: esp32-rs485.sch (EAGLE design)
At the start: 24 parts, among them J1 GREEN-2P-3.5, U1 TEXAS_INSTRUMENTS_TPS54360DDA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, U2 MAX3485CSA

Commit message: Add MAX3485, CH340K and associated passives
Add MAX3485 TTL serial to RS-485 transceiver and associated passives.
Add CH340K USB to TTL serial chip and associated passives, ESP reset circuitry and PCB edge USB-C connector (must use 0.8mm PCB).
Complete PCB layout.
Parts:
- removed J3: (no value), SparkFun-Connectors:6_PIN_SERIAL_TARGETSILK
- removed U$1: ESP32-PICO-D4, ESP32-PICO-D4:ESP32-PICO-D4
- added C11, C8, C9: 100nf, OPL_Capacitor:CERAMIC-100NF-25V-10%-X7R(0402)
- added C12: 1UF 6.3V, OPL_Capacitor:CERAMIC-1UF-6.3V-10%-X5R(0402)
- added R10, R9: 470R, OPL_Resistor:SMD-RES-470R-1%-1/16W(0402)
- added R11: 220R, OPL_Resistor:SMD-RES-270R-1%-1/16W(0402)
- added R7, R8: 10K 1/16W, OPL_Resistor:SMD-RES-10K-1%-1/16W(0402)
- added U$2: PCB_USB_C_2.0DS_2, USB_pcb_connectors:PCB_USB_C_2.0DS_2
- added U3: CH340K, CH340K:CH340K
- added U4: TPS54360, we-power:TPS54360
- U1: value TEXAS_INSTRUMENTS_TPS54360DDARTEXAS_INSTRUMENTS_TPS54360DDAR_0_0 -> ESP32-PICO-D4; device Texas Instruments - TPS54360DDAR:TEXAS_INSTRUMENTS_TPS54360DDARTEXAS_INSTRUMENTS_TPS54360DDAR_0_0 -> ESP32-PICO-D4:ESP32-PICO-D4
Connections:
- removed net N$5: C2.2, C3.2, F1.1, U1.VIN
- removed net N$7: C5.2, R2.2, U1.COMP
- new net +24V: C2.2, C3.2, F1.1, U4.VIN
- new net DTR: Q1Q1.E, R6.1, U3.DTR
- new net EN: C8.1, Q1Q2.C, R7.1, U1.EN
- new net GPIO0: Q1Q1.C, R8.1, U1.IO0
- new net N$10: R10.1, U3.TXD
- new net N$11: R9.1, U3.RXD
- new net N$12: U$2.D+, U3.USBDN
- new net N$13: U$2.D-, U3.USBDP
- new net N$14: C5.2, R2.2, U4.COMP
- new net N$3: Q1Q1.B, R5.2
- new net N$9: Q1Q2.B, R6.2
- new net RTS: Q1Q2.E, R5.1, U3.RTS
- new net U0RXD: R10.2, U1.U0RXD
- new net U0TXD: R9.2, U1.U0TXD
- net 3V3: now also C11.2, C12.2, C9.1, R7.2, R8.2, U1.IO21, U1.VDD3P3_CPU, U1.VDD3P3_RTC, U1.VDDA, U1.VDDA3P3_1, U1.VDDA_2, U1.VDDA_3, U1.VDDA_3P3, U1.XTAL_P_NC, U3.V3, U3.VCC; no longer U$1.VDDA, U$1.VDDA3P3_1, U$1.VDDA_3P3
- net A: now also R11.1
- net B: now also R11.2
- net FB: now also U4.FB; no longer U1.FB
- net GND: now also C11.1, C12.1, C8.2, C9.2, U$2.VBUS, U3.GND, U3.GND2, U4.GND; no longer J3.GND, U1.POWERPAD
- net N$1: now also U1.LNA_IN; no longer U$1.LNA_IN
- net N$2: now also U4.BOOT; no longer U1.BOOT
- net N$6: now also U4.RT_CLK; no longer U1.RT/CLK
- net SW: now also U4.SW; no longer U1.SW
- net U1RTS: now also U1.CMD; no longer U$1.CMD
- net U1RXD: now also U1.SD2; no longer U$1.SD2
- net U1TXD: now also U1.SD3; no longer U$1.SD3
Other:
- moved on the sheet: C1, C2, C3, C4, C5, Q1Q1, Q1Q2, R1, R2, R5, R6
